Commit message: ex2.1

File: src/my_box_bot_description/urdf/box_bot_meshes_collisions_inertias.urdf (robot description, URDF)
Before this commit: robot box_bot, 10 links, 9 joints
Links:
- link back_pitch_link: mass None -> 0.001; geometry collision sphere radius=0.010; visual sphere radius=0.010
- link back_roll_link: mass None -> 0.001; geometry collision cylinder length=0.001 radius=0.0045000000000000005; visual cylinder length=0.001 radius=0.0045000000000000005
- link back_yaw_link: mass None -> 0.001; geometry collision cylinder length=0.001 radius=0.0045000000000000005; visual cylinder length=0.001 radius=0.0045000000000000005
- link chassis: mass None -> 0.5; geometry collision box size=0.1 0.1 0.1; visual mesh filename=package://my_box_bot_description/meshes/cute_cube.dae scale=0.1 0.1 0.1
- link front_pitch_link: mass None -> 0.001; geometry collision sphere radius=0.010; visual sphere radius=0.010
- link front_roll_link: mass None -> 0.001; geometry collision cylinder length=0.001 radius=0.0045000000000000005; visual cylinder length=0.001 radius=0.0045000000000000005
- link front_yaw_link: mass None -> 0.001; geometry collision cylinder length=0.001 radius=0.0045000000000000005; visual cylinder length=0.001 radius=0.0045000000000000005
- link left_wheel: mass None -> 0.05; geometry collision cylinder length=0.001 radius=0.035; visual cylinder length=0.001 radius=0.035
- link right_wheel: mass None -> 0.05; geometry collision cylinder length=0.001 radius=0.035; visual cylinder length=0.001 radius=0.035
